File: JmpAperature/TestBoard1.brd (EAGLE design)
At the start: 160 x 100 mm, 4 parts

Commit message: updated
Parts:
- added SJ10, SJ13, SJ14, SJ17, SJ18, SJ21, SJ22, SJ25, SJ26, SJ29, SJ30, SJ5, SJ6, SJ9: JUMPER-PAD-2-NO, TestAperatures:PAD-JUMPER-2-NO_NO_SILK
- added SJ11, SJ12, SJ15, SJ16, SJ19, SJ20, SJ23, SJ24, SJ27, SJ28, SJ31, SJ32, SJ7, SJ8: JUMPER-PAD-3-NOYES_SILK, TestAperatures:PAD-JUMPER-3-NO_YES_SILK
- SJ1: value JUMPER-PAD-2-NC_BY_PASTE -> JUMPER-PAD-2-NO; device TestAperatures:PAD-JUMPER-2-NC_BY_PASTE_YES_SILK -> TestAperatures:PAD-JUMPER-2-NO_NO_SILK
- SJ2: value JUMPER-PAD-2-NC_BY_PASTEFULL-BOX-SILK -> JUMPER-PAD-2-NO; device TestAperatures:PAD-JUMPER-2-NC_BY_PASTE_YES_SILK_FULL_BOX -> TestAperatures:PAD-JUMPER-2-NO_NO_SILK
- SJ3: value JUMPER-PAD-3-2OF3_NC_BY_PASTE -> JUMPER-PAD-3-NOYES_SILK; device TestAperatures:PAD-JUMPER-3-2OF3_NC_BY_PASTE_YES_SILK_FULL_BOX -> TestAperatures:PAD-JUMPER-3-NO_YES_SILK
- SJ4: value JUMPER-PAD-3-NC_BY_PASTE -> JUMPER-PAD-3-NOYES_SILK; device TestAperatures:PAD-JUMPER-3-NC_BY_PASTE_YES_SILK_FULL_BOX -> TestAperatures:PAD-JUMPER-3-NO_YES_SILK
- moved SJ4 11.7 mm to (21.6, 16.5), turned to 90 degrees
- moved SJ2 10.2 mm to (21.6, 21.6)
- moved SJ1 8.52 mm to (16.5, 21.6), turned to 0 degrees
- moved SJ3 5.08 mm to (16.5, 16.5), turned to 0 degrees
Connections:
- removed net GND: SJ1.1, SJ2.1, SJ3.3, SJ4.3
- removed net PWR: SJ1.2, SJ2.2, SJ3.1, SJ4.1
Routing:
- net GND: track 23.0 -> 0.00 mm
- net PWR: track 22.9 -> 0.00 mm
- added copper zone on layer 1, net GND
Other:
- board size 160 x 100 mm -> 165.1 x 101.6 mm
- board text added: "10%"
- board text added: "20%"
- board text added: "30%"
- board text added: "40%"
- board text added: "50%"
- board text added: "60%"
- board text added: "70%"
- board text added: "Control"

Commit message: First row plus footprints
Parts:
- added SJ100, SJ103, SJ104, SJ107, SJ108, SJ111, SJ112, SJ115, SJ116, SJ119, SJ120, SJ123, SJ124, SJ127, SJ128, SJ131, SJ132, SJ135, SJ136, SJ139, SJ140, SJ143, SJ144, SJ147, SJ148, SJ151, SJ152, SJ155, SJ156, SJ159, SJ160, SJ163, SJ164, SJ35, SJ36, SJ39, SJ40, SJ43, SJ44, SJ47, SJ48, SJ51, SJ52, SJ55, SJ56, SJ59, SJ60, SJ63, SJ64, SJ67, SJ68, SJ71, SJ72, SJ75, SJ76, SJ79, SJ80, SJ83, SJ84, SJ87, SJ88, SJ91, SJ92, SJ95, SJ96, SJ99: JUMPER-PAD-3-NOYES_SILK, TestAperatures:PAD-JUMPER-3-NO_YES_SILK
- added SJ101, SJ102, SJ105, SJ106, SJ109, SJ110, SJ113, SJ114, SJ117, SJ118, SJ121, SJ122, SJ125, SJ126, SJ129, SJ130, SJ133, SJ134, SJ137, SJ138, SJ141, SJ142, SJ145, SJ146, SJ149, SJ150, SJ153, SJ154, SJ157, SJ158, SJ161, SJ162, SJ33, SJ34, SJ37, SJ38, SJ41, SJ42, SJ45, SJ46, SJ49, SJ50, SJ53, SJ54, SJ57, SJ58, SJ61, SJ62, SJ65, SJ66, SJ69, SJ70, SJ73, SJ74, SJ77, SJ78, SJ81, SJ82, SJ85, SJ86, SJ89, SJ90, SJ93, SJ94, SJ97, SJ98: JUMPER-PAD-2-NO, TestAperatures:PAD-JUMPER-2-NO_NO_SILK
- moved SJ29 149.5 mm to (0.00, -50.8)
- moved SJ30 148.9 mm to (12.7, -50.8), turned to 0 degrees
- moved SJ26 140.1 mm to (-12.7, -50.8), turned to 0 degrees
- moved SJ25 125.1 mm to (38.1, -38.1)
- moved SJ31 121.7 mm to (-12.7, -25.4)
- moved SJ32 120.1 mm to (0.00, -25.4), turned to 0 degrees
- moved SJ21 110.6 mm to (12.7, -38.1)
- moved SJ22 110.6 mm to (25.4, -38.1), turned to 0 degrees
- moved SJ27 92.8 mm to (12.7, -12.7)
- moved SJ28 92.8 mm to (25.4, -12.7), turned to 0 degrees
- moved SJ23 85.2 mm to (-12.7, -12.7)
- moved SJ24 82.9 mm to (0.00, -12.7), turned to 0 degrees
