File: USBSolder/USBSolder.sch (EAGLE design)
At the start: 13 parts

Commit message: done with usb test
Parts:
- removed JP3, JP5: (no value), TestUSBs:USB_MICROB_PLUG
- added JP13, JP14: (no value), TestUSBs:USB_MICROB_PLUGCONN-11752
- JP1, JP11, JP7, JP9: device SparkFun-Connectors:USB_MICROB_PLUGCONN-11752 -> TestUSBs:USB_MICROB_PLUGCONN-11752
Connections:
- net 5V1: now also JP14.VCC; no longer JP5.VCC
- net GND: now also JP13.GND, JP14.GND; no longer JP3.GND, JP5.GND
- net N$10: now also JP13.VCC; no longer JP3.VCC
Changed lines of the file:
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@@
 <parts>
 <part name="FRAME1" library="SparkFun-Aesthetics" deviceset="FRAME-LETTER" device=""/>
-<part name="JP1" library="SparkFun-Connectors" deviceset="USB_MICROB_PLUG" device="CONN-11752"/>
+<part name="JP1" library="TestUSBs" deviceset="USB_MICROB_PLUG" device="CONN-11752"/>
 <part name="JP2" library="SparkFun-Connectors" deviceset="M05" device="PTH"/>
 <part name="GND1" library="SparkFun-Aesthetics" deviceset="GND" device=""/>
-<part name="JP3" library="TestUSBs" deviceset="USB_MICROB_PLUG" device=""/>
 <part name="JP4" library="SparkFun-Connectors" deviceset="M05" device="PTH"/>
 <part name="GND2" library="SparkFun-Aesthetics" deviceset="GND" device=""/>
-<part name="JP5" library="TestUSBs" deviceset="USB_MICROB_PLUG" device=""/>
 <part name="JP6" library="SparkFun-Connectors" deviceset="M05" device="PTH"/>
 <part name="GND3" library="SparkFun-Aesthetics" deviceset="GND" device=""/>
-<part name="JP7" library="SparkFun-Connectors" deviceset="USB_MICROB_PLUG" device="CONN-11752"/>
+<part name="JP7" library="TestUSBs" deviceset="USB_MICROB_PLUG" device="CONN-11752"/>
 <part name="JP8" library="SparkFun-Connectors" deviceset="M05" device="PTH"/>
 <part name="GND4" library="SparkFun-Aesthetics" deviceset="GND" device=""/>
-<part name="JP9" library="SparkFun-Connectors" deviceset="USB_MICROB_PLUG" device="CONN-11752"/>
+<part name="JP9" library="TestUSBs" deviceset="USB_MICROB_PLUG" device="CONN-11752"/>
 <part name="JP10" library="SparkFun-Connectors" deviceset="M05" device="PTH"/>
 <part name="GND5" library="SparkFun-Aesthetics" deviceset="GND" device=""/>
-<part name="JP11" library="SparkFun-Connectors" deviceset="USB_MICROB_PLUG" device="CONN-11752"/>
+<part name="JP11" library="TestUSBs" deviceset="USB_MICROB_PLUG" device="CONN-11752"/>
 <part name="JP12" library="SparkFun-Connectors" deviceset="M05" device="PTH"/>
 <part name="GND6" library="SparkFun-Aesthetics" deviceset="GND" device=""/>
 <part name="GND7" library="SparkFun-Aesthetics" deviceset="GND" device=""/>
+<part name="JP13" library="TestUSBs" deviceset="USB_MICROB_PLUG" device="CONN-11752"/>
+<part name="JP14" library="TestUSBs" deviceset="USB_MICROB_PLUG" device="CONN-11752"/>
 </parts>
 <sheets>
@@
 <instance part="JP2" gate="G$1" x="12.7" y="152.4"/>
 <instance part="GND1" gate="1" x="43.18" y="147.32"/>
-<instance part="JP3" gate="G$1" x="71.12" y="152.4"/>
 <instance part="JP4" gate="G$1" x="50.8" y="152.4"/>
 <instance part="GND2" gate="1" x="60.96" y="142.24"/>
-<instance part="JP5" gate="G$1" x="109.22" y="152.4"/>
 <instance part="JP6" gate="G$1" x="88.9" y="152.4"/>
 <instance part="GND3" gate="1" x="99.06" y="142.24"/>
@@
 <instance part="GND6" gate="1" x="238.76" y="147.32"/>
 <instance part="GND7" gate="1" x="218.44" y="142.24"/>
+<instance part="JP13" gate="G$1" x="71.12" y="152.4"/>
+<instance part="JP14" gate="G$1" x="109.22" y="152.4"/>
 </instances>
 <busses>
@@
 </segment>
 <segment>
-<pinref part="JP3" gate="G$1" pin="GND"/>
 <pinref part="JP4" gate="G$1" pin="1"/>
 <wire x1="58.42" y1="147.32" x2="60.96" y2="147.32" width="0.1524" layer="91"/>
@@
 <wire x1="60.96" y1="147.32" x2="63.5" y2="147.32" width="0.1524" layer="91"/>
 <junction x="60.96" y="147.32"/>
-</segment>
-<segment>
-<pinref part="JP5" gate="G$1" pin="GND"/>
+<pinref part="JP13" gate="G$1" pin="GND"/>
+</segment>
+<segment>
 <pinref part="JP6" gate="G$1" pin="1"/>
 <wire x1="96.52" y1="147.32" x2="99.06" y2="147.32" width="0.1524" layer="91"/>
@@
 <junction x="99.06" y="147.32"/>
 <pinref part="GND3" gate="1" pin="GND"/>
+<pinref part="JP14" gate="G$1" pin="GND"/>
 </segment>
 <segment>
@@
 <net name="N$10" class="0">
 <segment>
-<pinref part="JP3" gate="G$1" pin="VCC"/>
 <pinref part="JP4" gate="G$1" pin="5"/>
 <wire x1="58.42" y1="157.48" x2="63.5" y2="157.48" width="0.1524" layer="91"/>
+<pinref part="JP13" gate="G$1" pin="VCC"/>
 </segment>
 </net>
 <net name="5V1" class="0">
 <segment>
-<pinref part="JP5" gate="G$1" pin="VCC"/>
 <pinref part="JP6" gate="G$1" pin="5"/>
 <wire x1="96.52" y1="157.48" x2="101.6" y2="157.48" width="0.1524" layer="91"/>
+<pinref part="JP14" gate="G$1" pin="VCC"/>
 </segment>
 </net>
@@
 </sheet>
 </sheets>
+<errors>
+</errors>
 </schematic>
 </drawing>
