File: JmpAperture/TestBoardExport.brd (EAGLE design)
At the start: 108 x 69.8 mm, 380 parts

Commit message: touch-ups
Parts:
- SJ21, SJ22, SJ23, SJ24: value JUMPER-PAD-3-NOYES_SILK -> JUMPER-PAD-3-NO3_0; device TestAperatures:PAD-JUMPER-3-NO_YES_SILK -> TestAperatures:PAD-JUMPER-3-NO_YES_SILK_ALL
- SJ73, SJ74, SJ75, SJ76: value JUMPER-PAD-3-NOYES_SILK -> JUMPER-PAD-3-NO3_20; device TestAperatures:PAD-JUMPER-3-NO_YES_SILK -> TestAperatures:PAD-JUMPER-3-NO_YES_SILK_ALL_20

Commit message: added example shapes for dfm
Parts:
- moved SJ155 6.99 mm to (19.7, 47.0)
- moved SJ195 6.99 mm to (19.7, 59.7)
- moved SJ127 6.67 mm to (22.5, 47.0)
- moved SJ167 6.67 mm to (22.5, 59.7)
- moved SJ156 6.36 mm to (21.6, 43.5)
- moved SJ196 6.36 mm to (21.6, 56.2)
- moved C101 6.35 mm to (92.7, 32.7)
- moved C103 6.35 mm to (96.5, 30.8)
- moved C104 6.35 mm to (99.4, 33.7)
- moved C105 6.35 mm to (83.8, 36.2)
- moved C106 6.35 mm to (84.5, 31.1)
- moved C129 6.35 mm to (66.7, 45.4)
- moved C131 6.35 mm to (74.6, 45.7)
- moved C132 6.35 mm to (71.8, 40.3)
- moved C135 6.35 mm to (87.6, 46.4)
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Other:
- board size 108 x 69.8 mm -> 107.9 x 69.8 mm
