File: JmpAperture/TestBoardExport.sch (EAGLE design)
At the start: 380 parts

Commit message: touch-ups
Parts:
- SJ21, SJ22, SJ23, SJ24: value JUMPER-PAD-3-NOYES_SILK -> JUMPER-PAD-3-NO3_0; device TestAperatures:JUMPER-PAD-3-NOYES_SILK -> TestAperatures:JUMPER-PAD-3-NO3_0
- SJ73, SJ74, SJ75, SJ76: value JUMPER-PAD-3-NOYES_SILK -> JUMPER-PAD-3-NO3_20; device TestAperatures:JUMPER-PAD-3-NOYES_SILK -> TestAperatures:JUMPER-PAD-3-NO3_20
Changed lines of the file:
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@@
 <part name="GND15" library="SparkFun-Aesthetics" deviceset="GND" device=""/>
 <part name="GND16" library="SparkFun-Aesthetics" deviceset="GND" device=""/>
-<part name="SJ21" library="TestAperatures" deviceset="JUMPER-PAD-3-NO" device="YES_SILK"/>
-<part name="SJ22" library="TestAperatures" deviceset="JUMPER-PAD-3-NO" device="YES_SILK"/>
-<part name="SJ23" library="TestAperatures" deviceset="JUMPER-PAD-3-NO" device="YES_SILK"/>
-<part name="SJ24" library="TestAperatures" deviceset="JUMPER-PAD-3-NO" device="YES_SILK"/>
+<part name="SJ21" library="TestAperatures" deviceset="JUMPER-PAD-3-NO" device="3_0" value="JUMPER-PAD-3-NO3_0"/>
+<part name="SJ22" library="TestAperatures" deviceset="JUMPER-PAD-3-NO" device="3_0" value="JUMPER-PAD-3-NO3_0"/>
+<part name="SJ23" library="TestAperatures" deviceset="JUMPER-PAD-3-NO" device="3_0" value="JUMPER-PAD-3-NO3_0"/>
+<part name="SJ24" library="TestAperatures" deviceset="JUMPER-PAD-3-NO" device="3_0" value="JUMPER-PAD-3-NO3_0"/>
 <part name="SJ25" library="TestAperatures" deviceset="JUMPER-PAD-3-NO" device="3_0" value="JUMPER-PAD-3-NO3_0"/>
 <part name="SJ26" library="TestAperatures" deviceset="JUMPER-PAD-3-NO" device="3_0" value="JUMPER-PAD-3-NO3_0"/>
@@
 <part name="GND31" library="SparkFun-Aesthetics" deviceset="GND" device=""/>
 <part name="GND32" library="SparkFun-Aesthetics" deviceset="GND" device=""/>
-<part name="SJ73" library="TestAperatures" deviceset="JUMPER-PAD-3-NO" device="YES_SILK"/>
-<part name="SJ74" library="TestAperatures" deviceset="JUMPER-PAD-3-NO" device="YES_SILK"/>
-<part name="SJ75" library="TestAperatures" deviceset="JUMPER-PAD-3-NO" device="YES_SILK"/>
-<part name="SJ76" library="TestAperatures" deviceset="JUMPER-PAD-3-NO" device="YES_SILK"/>
+<part name="SJ73" library="TestAperatures" deviceset="JUMPER-PAD-3-NO" device="3_20" value="JUMPER-PAD-3-NO3_20"/>
+<part name="SJ74" library="TestAperatures" deviceset="JUMPER-PAD-3-NO" device="3_20" value="JUMPER-PAD-3-NO3_20"/>
+<part name="SJ75" library="TestAperatures" deviceset="JUMPER-PAD-3-NO" device="3_20" value="JUMPER-PAD-3-NO3_20"/>
+<part name="SJ76" library="TestAperatures" deviceset="JUMPER-PAD-3-NO" device="3_20" value="JUMPER-PAD-3-NO3_20"/>
 <part name="SJ77" library="TestAperatures" deviceset="JUMPER-PAD-3-NO" device="3_20" value="JUMPER-PAD-3-NO3_20"/>
 <part name="SJ78" library="TestAperatures" deviceset="JUMPER-PAD-3-NO" device="3_20" value="JUMPER-PAD-3-NO3_20"/>
